File: Latch Circuit/LatchCircuit.kicad_pcb (KiCad board)
At the start: 2 copper layers, 0 parts

Commit message: update schematic; add WIP pcb
Parts:
- added C1: 10u, Capacitor_THT:CP_Radial_D5.0mm_P2.00mm, F.Cu at (43.9, 45.7)
- added C2: 100n, Capacitor_SMD:C_0603_1608Metric_Pad1.08x0.95mm_HandSolder, F.Cu at (55.9, 51.6)
- added C3: 100n, Capacitor_SMD:C_0603_1608Metric_Pad1.08x0.95mm_HandSolder, F.Cu at (50.3, 38.9)
- added C4: 100n, Capacitor_SMD:C_0603_1608Metric_Pad1.08x0.95mm_HandSolder, F.Cu at (41.9, 51.5)
- added D1: BAT54W, Package_TO_SOT_SMD:SOT-323_SC-70, F.Cu at (45.2, 75.2)
- added D2: BAT54W, Package_TO_SOT_SMD:SOT-323_SC-70, F.Cu at (64.8, 35.9)
- added D3: LED, LED_SMD:LED_0805_2012Metric_Pad1.15x1.40mm_HandSolder, F.Cu at (45.0, 70.1)
- added D4: LED, LED_SMD:LED_0805_2012Metric_Pad1.15x1.40mm_HandSolder, F.Cu at (50.0, 65.5)
- added D5: LED, LED_SMD:LED_0805_2012Metric_Pad1.15x1.40mm_HandSolder, F.Cu at (27.7, 71.6)
- added H1: MountingHole, MountingHole:MountingHole_2.2mm_M2, F.Cu at (37.3, 75.9)
- added H2: MountingHole, MountingHole:MountingHole_2.2mm_M2, F.Cu at (40.9, 39.1)
- added H3: MountingHole, MountingHole:MountingHole_2.2mm_M2, F.Cu at (66.3, 29.0)
- added H4: MountingHole, MountingHole:MountingHole_2.2mm_M2, F.Cu at (29.5, 75.9)
- added J1: 12V_Power, Connector_Molex:Molex_Micro-Fit_3.0_43650-0200_1x02_P3.00mm_Horizontal, F.Cu at (34.2, 65.5)
- added J2: IMD_AMS, Connector_Molex:Molex_Micro-Fit_3.0_43650-0200_1x02_P3.00mm_Horizontal, F.Cu at (60.5, 45.5)
- added J3: ExternalLEDs, Connector_Molex:Molex_Micro-Fit_3.0_43650-0200_1x02_P3.00mm_Horizontal, F.Cu at (60.5, 68.3)
- added J4: Shutdown, Connector_Molex:Molex_Micro-Fit_3.0_43650-0200_1x02_P3.00mm_Horizontal, F.Cu at (34.5, 30.7)
- added K1: G5Q-1EU DC12, Relay_THT:Relay_SPDT_Omron-G5Q-1, F.Cu at (34.5, 55.6)
- added K2: G5Q-1EU DC12, Relay_THT:Relay_SPDT_Omron-G5Q-1, F.Cu at (60.2, 25.7)
- added Q1: XP262N7002TR-G, Package_TO_SOT_SMD:SOT-23, F.Cu at (40.9, 65.3)
- added Q2: XP262N7002TR-G, Package_TO_SOT_SMD:SOT-23, F.Cu at (58.9, 38.6)
- added R1: 10k, Resistor_SMD:R_0603_1608Metric_Pad0.98x0.95mm_HandSolder, F.Cu at (36.3, 70.9)
- added R2: 10k, Resistor_SMD:R_0603_1608Metric_Pad0.98x0.95mm_HandSolder, F.Cu at (46.5, 38.9)
- added R3: 1k, Resistor_SMD:R_0603_1608Metric_Pad0.98x0.95mm_HandSolder, F.Cu at (39.9, 69.8)
- added R4: 1k, Resistor_SMD:R_0603_1608Metric_Pad0.98x0.95mm_HandSolder, F.Cu at (54.6, 65.3)
- added R5: 10k, Resistor_SMD:R_0603_1608Metric_Pad0.98x0.95mm_HandSolder, F.Cu at (45.7, 65.5)
- added R6: 1k, Resistor_SMD:R_0603_1608Metric_Pad0.98x0.95mm_HandSolder, F.Cu at (31.8, 70.9)
- added SW1: Reset, Connector_Molex:Molex_Micro-Fit_3.0_43650-0200_1x02_P3.00mm_Horizontal, F.Cu at (60.5, 56.9)
- added U1: 4013, Package_SO:SOIC-14_3.9x8.7mm_P1.27mm, F.Cu at (53.0, 58.0)
- added U2: 40106, Package_SO:SOIC-14_3.9x8.7mm_P1.27mm, F.Cu at (52.6, 46.0)
- added U3: 4013, Package_SO:SOIC-14_3.9x8.7mm_P1.27mm, F.Cu at (42.7, 57.1)
- added U5: 40106, Package_SO:SOIC-14_3.9x8.7mm_P1.27mm, F.Cu at (51.8, 73.7)
Routing:
- net GND: track 0.00 -> 93.8 mm, vias 0 -> 11
- net /IMD_FAULT_LATCHED: track 0.00 -> 66.1 mm, vias 0 -> 2
- net /~{AMS_NO_FAULT}: track 0.00 -> 36.2 mm, vias 0 -> 2
- net Net-(U1-Pad6): track 0.00 -> 30.4 mm, vias 0 -> 2
- net Net-(D1-Pad1): track 0.00 -> 29.0 mm
- net /POR: track 0.00 -> 28.4 mm
- net Net-(U3-Pad6): track 0.00 -> 24.5 mm, vias 0 -> 2
- net /AMS_FAULT_LATCHED: track 0.00 -> 23.6 mm
- net Net-(C1-Pad1): track 0.00 -> 21.3 mm
- net Net-(K1-Pad3): track 0.00 -> 20.5 mm
- net /SHUTDOWN_OUT: track 0.00 -> 19.2 mm
- net Net-(D2-Pad1): track 0.00 -> 18.6 mm
- net +12V: track 0.00 -> 18.5 mm
- net /IMD_OK_{HS}: track 0.00 -> 10.3 mm
- net /SHUTDOWN_IN: track 0.00 -> 10.0 mm
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- added copper zone on F.Cu, net +12V
- added copper zone on B.Cu, net GND
Other:
- board outline added: 45.7 x 55.9 mm
